File: hardware/fpanel_remote_pcb_v1/fpanel_remote_pcb.kicad_sch (KiCad schematic)
At the start: 20 parts, among them J1 Conn_02x04_Odd_Even, J2 Conn_02x04_Odd_Even, J3 PS/2 HDR, U1 pi_pico_w, U2 SSM6N44FE, U3 SSM6N44FE, U4 SSM6N44FE

Commit message: fix pcb and schematics
Parts:
- R1, R11, R2, R5: value 100K -> 10K
- R10, R6, R7, R9: value 200K -> 10K
Connections:
- net GND: now also U4.1 (Q1_S), U4.4 (Q2_S); no longer U4.3 (Q2_D), U4.6 (Q1_D)
- net PS2_CLK: now also U4.6 (Q1_D); no longer U4.1 (Q1_S)
- net PS2_DATA: now also U4.3 (Q2_D); no longer U4.4 (Q2_S)
- net at J1.5 (Pin_5), J2.5 (Pin_5): now also U2.3 (Q2_D); no longer U2.4 (Q2_S), U2.6 (Q1_D)
- net at J1.6 (Pin_6), J2.6 (Pin_6): now also U3.3 (Q2_D); no longer U3.4 (Q2_S), U3.6 (Q1_D)
- net at J1.7 (Pin_7), J2.7 (Pin_7): now also U2.6 (Q1_D); no longer U2.1 (Q1_S), U2.3 (Q2_D)
- net at J1.8 (Pin_8), J2.8 (Pin_8): now also U3.6 (Q1_D); no longer U3.1 (Q1_S), U3.3 (Q2_D)
- new net: U2.1 (Q1_S), U2.4 (Q2_S)
- new net: U3.1 (Q1_S), U3.4 (Q2_S)
Other:
- moved on the sheet: R3, R4
