File: hardware/fpanel_remote_pcb_v1/fpanel_remote_pcb.kicad_pcb (KiCad board)
At the start: 2 copper layers, 45.7 x 53.3 mm, 20 parts, among them J1 Conn_02x04_Odd_Even, J2 Conn_02x04_Odd_Even, J3 PS/2 HDR, U1 pi_pico_w, U2 SSM6N44FE, U3 SSM6N44FE, U4 SSM6N44FE

Commit message: fix pcb and schematics
Parts:
- R1, R11, R2, R5: value 100K -> 10K
- R10, R6, R7, R9: value 200K -> 10K
- turned R2 to 90 degrees
- turned R5 to -90 degrees
Connections:
- J1 pad 5: Net-(U2-Pad4) -> Net-(J1-Pin_5)
- J1 pad 6: Net-(U3-Pad4) -> Net-(J1-Pin_6)
- J1 pad 7: Net-(U2-Pad1) -> Net-(J1-Pin_7)
- J1 pad 8: Net-(U3-Pad1) -> Net-(J1-Pin_8)
- J2 pad 5: Net-(U2-Pad4) -> Net-(J1-Pin_5)
- J2 pad 6: Net-(U3-Pad4) -> Net-(J1-Pin_6)
- J2 pad 7: Net-(U2-Pad1) -> Net-(J1-Pin_7)
- J2 pad 8: Net-(U3-Pad1) -> Net-(J1-Pin_8)
- U2 pad 1: Net-(U2-Pad1) -> Net-(U2-Q1_S)
- U2 pad 3: Net-(U2-Pad1) -> Net-(J1-Pin_5)
- U2 pad 4: Net-(U2-Pad4) -> Net-(U2-Q1_S)
- U2 pad 6: Net-(U2-Pad4) -> Net-(J1-Pin_7)
- U3 pad 1: Net-(U3-Pad1) -> Net-(U3-Q1_S)
- U3 pad 3: Net-(U3-Pad1) -> Net-(J1-Pin_6)
- U3 pad 4: Net-(U3-Pad4) -> Net-(U3-Q1_S)
- U3 pad 6: Net-(U3-Pad4) -> Net-(J1-Pin_8)
- U4 pad 1: PS2_CLK -> GND
- U4 pad 3: GND -> PS2_DATA
- U4 pad 4: PS2_DATA -> GND
- U4 pad 6: GND -> PS2_CLK
Routing:
- net Net-(U3-Pad1): track 46.4 -> 0.00 mm, vias 2 -> 0
- net Net-(J1-Pin_6): track 0.00 -> 36.6 mm, vias 0 -> 2
- net Net-(U2-Pad1): track 35.1 -> 0.00 mm, vias 3 -> 0
- net Net-(U2-Pad4): track 31.6 -> 0.00 mm, vias 4 -> 0
- net Net-(J1-Pin_8): track 0.00 -> 31.4 mm, vias 0 -> 2
- net Net-(J1-Pin_5): track 0.00 -> 29.4 mm, vias 0 -> 4
- net Net-(U3-Pad4): track 29.2 -> 0.00 mm
- net Net-(J1-Pin_7): track 0.00 -> 28.9 mm, vias 0 -> 5
- net Net-(U3-Q1_S): track 0.00 -> 4.69 mm, vias 0 -> 2
- net RESET_SW: track 30.1 -> 34.5 mm
- net Net-(U2-Q1_S): track 0.00 -> 4.37 mm, vias 0 -> 2
- net PI_PS2_DATA: track 60.6 -> 56.3 mm
- net PI_PS2_CLK: track 56.8 -> 52.8 mm
- net PS2_CLK: track 15.1 -> 18.1 mm
- net GND: track 50.3 -> 52.9 mm, vias 18 -> 17
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
Commit message: update pcb - minor changes
Other:
- board text added: "COOLHORSE INDUSTRIES (C) 2023"
- board text removed: "COOLHORSE INDUSTRIES (C) 2022"
Changed lines of the file:
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@@
       (drillshape 0)
       (scaleselection 1)
-      (outputdirectory "gerbers/")
+      (outputdirectory "fpanel_remote_gerbers/")
     )
   )
@@
     (effects (font (size 1 1) (thickness 0.15)) (justify mirror))
   )
-  (gr_text "COOLHORSE INDUSTRIES (C) 2022" (at 125.476 84.836 270) (layer "B.SilkS")
+  (gr_text "COOLHORSE INDUSTRIES (C) 2023" (at 125.476 84.836 270) (layer "B.SilkS")
     (effects (font (size 1 1) (thickness 0.15)) (justify mirror))
   )
